File: hw/sch_pcb/LED7SEG02.kicad_sch (KiCad schematic)
At the start: 16 parts, among them J1 Conn_02x05_Odd_Even, J4 DBG, SW1 MSSR-16S-TR, U1 STM32G031F8Px

Commit message: Correct project documentation structure.
Other:
- company: (none) -> Mlab.cz
- title: (none) -> LED7SEG02A
